File: libraries/G_SmartPiezo/Piezo.sch (EAGLE design)
At the start: 7 parts, among them U1 ATMEGA328

Commit message: The latest version of the module's eagle files
Parts:
- added R3, R4, R5: 10K, rcl:R-US_R0603
- R1: device SparkFun:RESISTOR-ARRAY0603-ARV -> rcl:R-US_R0603
Connections:
- net DN: now also R5.1; no longer R1C.2
- net N$1: now also R1.1; no longer R1B.1
- net N$2: now also R3.1; no longer R1A.1
- net SCL: now also R1.2; no longer R1B.2
- net SDA: now also R3.2; no longer R1A.2
- net UP: now also R4.1; no longer R1D.1
- net VCC: now also R4.2, R5.2; no longer R1C.1, R1D.2
Other:
- note removed: "DN"
- note removed: "MISO"
- note removed: "MOSI"
- note removed: "RST"
- note removed: "RX"
- note removed: "SCK"
- note removed: "SCL"
- note removed: "SDA"
- note removed: "SP1"
- note removed: "SP2"
- note removed: "TX"
- note removed: "UP"
